File: schematic/schematic.kicad_sch (KiCad schematic)
At the start: 8 parts

Commit message: Add boost converter
Parts:
- added U?: Boost_converter, symbol New_Library:Boost_converter
Connections:
- net GND: now also U?.1 (Vin-); no longer U?.10 (PGND2), U?.3 (PGND1), U?.4 (PGND1), U?.9 (PGND2)
- net at U?.13 (VM2), U?.14 (VM3), U?.24 (VM1): now also U?.4 (Vout+); no longer BT?.1 (+)
- new net: BT?.1 (+), U?.2 (Vin+)
- new net: U?.10 (PGND2), U?.3 (PGND1), U?.3 (Vout-), U?.4 (PGND1), U?.9 (PGND2)
Other:
- moved on the sheet: BT?
